File: microdronesmd.sch (EAGLE design)
At the start: 22 parts, among them Q1 SUP75N06-08, Q2 SUP75N06-08, Q3 SUP75N06-08, Q4 SUP75N06-08

Commit message: Second commit
Parts:
- removed Q4: SUP75N06-08, transistor-fet:SUP75N06-08
- added Q5: FDD4141TO252, transistor-fet:FDD4141TO252
- Q1, Q2, Q3: value SUP75N06-08 -> FDD4141TO252; device transistor-fet:SUP75N06-08 -> transistor-fet:FDD4141TO252
Connections:
- removed net GND: ARDUINO_NANO1.GND@2, BATTERY110-2.S, BATTERY350-2.S, BLUETOOTH.4, C1.2, MPU6050.7, Q1.S, Q2.S, Q3.S, Q4.S, R1.1, R2.1, R3.1, R4.1, R5.1, R6.1, R7.1
- new net GND/VCC: ARDUINO_NANO1.GND@2, BATTERY110-2.S, BATTERY350-2.S, BLUETOOTH.4, C1.2, MPU6050.7, Q1.G, Q2.G, Q3.G, Q5.G, R1.1, R2.1, R3.1, R4.1, R5.1, R6.1, R7.1
- net MOTOR1: now also Q5.D; no longer Q2.D
- net MOTOR3: now also Q2.D; no longer Q3.D
- net MOTOR4: now also Q3.D; no longer Q4.D
- net NPN1: now also Q5.S; no longer Q2.G
- net NPN2: now also Q1.S; no longer Q1.G
- net NPN3: now also Q2.S; no longer Q3.G
- net NPN4: now also Q3.S; no longer Q4.G
Other:
- moved on the sheet: ARDUINO_NANO1, BATTERY110-1, BATTERY110-2, BATTERY350-1, BATTERY350-2, BLUETOOTH, C1, MOTOR1-1, MOTOR1-2, MOTOR2-1, MOTOR2-2, MOTOR3-1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
